File: ha_plattform.sch (KiCad schematic (older format))
At the start: 12 parts, among them J3 Raspberry_Pi_2_3

Commit message: Changed track width, improved routing
Parts:
- IR_D1, IR_D2: footprint Diode_THT:D_A-405_P2.54mm_Vertical_KathodeUp -> Connector_PinHeader_2.54mm:PinHeader_1x02_P2.54mm_Vertical
- LDR1: footprint Connector_PinHeader_1.27mm:PinHeader_1x02_P1.27mm_Vertical -> Resistor_THT:R_Axial_DIN0204_L3.6mm_D1.6mm_P5.08mm_Horizontal
- R10k1: footprint Connector_PinHeader_1.27mm:PinHeader_1x02_P1.27mm_Vertical -> Resistor_THT:R_Axial_DIN0204_L3.6mm_D1.6mm_P7.62mm_Horizontal
Changed lines of the file:
@@
 F 0 "IR_D1" H 5120 1470 50  0000 L CNN
 F 1 "IRL81A" H 5060 1290 50  0000 C CNN
-F 2 "Diode_THT:D_A-405_P2.54mm_Vertical_KathodeUp" H 5100 1575 50  0001 C CNN
+F 2 "Connector_PinHeader_2.54mm:PinHeader_1x02_P2.54mm_Vertical" H 5100 1575 50  0001 C CNN
 F 3 "" H 5050 1400 50  0001 C CNN
 	1    5100 1400
@@
 F 0 "IR_D2" H 5620 1470 50  0000 L CNN
 F 1 "IRL81A" H 5560 1290 50  0000 C CNN
-F 2 "Diode_THT:D_A-405_P2.54mm_Vertical_KathodeUp" H 5600 1575 50  0001 C CNN
+F 2 "Connector_PinHeader_2.54mm:PinHeader_1x02_P2.54mm_Vertical" H 5600 1575 50  0001 C CNN
 F 3 "" H 5550 1400 50  0001 C CNN
 	1    5600 1400
@@
 F 0 "R10k1" V 4830 1600 50  0000 C CNN
 F 1 "R10k" V 4750 1600 50  0000 C CNN
-F 2 "Connector_PinHeader_1.27mm:PinHeader_1x02_P1.27mm_Vertical" V 4680 1600 50  0001 C CNN
+F 2 "Resistor_THT:R_Axial_DIN0204_L3.6mm_D1.6mm_P7.62mm_Horizontal" V 4680 1600 50  0001 C CNN
 F 3 "" H 4750 1600 50  0001 C CNN
 	1    4750 1600
@@
 F 0 "LDR1" H 8270 1746 50  0000 L CNN
 F 1 "LDR03" H 8270 1655 50  0000 L CNN
-F 2 "Connector_PinHeader_1.27mm:PinHeader_1x02_P1.27mm_Vertical" V 8375 1700 50  0001 C CNN
+F 2 "Resistor_THT:R_Axial_DIN0204_L3.6mm_D1.6mm_P5.08mm_Horizontal" V 8375 1700 50  0001 C CNN
 F 3 "http://www.elektronica-componenten.nl/WebRoot/StoreNL/Shops/61422969/54F1/BA0C/C664/31B9/2173/C0A8/2AB9/2AEF/LDR03IMP.pdf" H 8200 1650 50  0001 C CNN
 	1    8200 1700

Commit message: fixed layout issues. moved led to front. rerouted whole board
Parts:
- removed IR_Input1: TSOP382xx, Package_TO_SOT_THT:TO-220-3_Vertical, symbol ha_plattform-rescue:TSOP382xx
- added R56_1: R, Resistor_THT:R_Axial_DIN0204_L3.6mm_D1.6mm_P7.62mm_Horizontal, symbol Device:R
- added U1: TSOP45xx_0, Package_TO_SOT_THT:TO-220-3_Vertical, symbol tsdp48xx_0:TSOP45xx_0
- C_0.22F1: footprint Capacitor_THT:CP_Radial_D10.0mm_P5.00mm -> Capacitor_THT:CP_Radial_D14.0mm_P5.00mm
Connections:
- wire segments 94 -> 101

Commit message: reduced footprint for capacitor
Parts:
- C_0.22F1: footprint Capacitor_THT:CP_Radial_D14.0mm_P5.00mm -> Capacitor_THT:CP_Radial_D10.0mm_P5.00mm
- renumbered U1 to TSOP48xx_1
Changed lines of the file:
@@
 F 0 "C_0.22F1" H 8318 2146 50  0000 L CNN
 F 1 "0.22F" H 8318 2055 50  0000 L CNN
-F 2 "Capacitor_THT:CP_Radial_D14.0mm_P5.00mm" H 8238 1950 50  0001 C CNN
+F 2 "Capacitor_THT:CP_Radial_D10.0mm_P5.00mm" H 8238 1950 50  0001 C CNN
 F 3 "~" H 8200 2100 50  0001 C CNN
 	1    8200 2100
@@
 	6400 3100 6400 5000
 $Comp
-L tsdp48xx_0:TSOP45xx_0 U1
+L tsdp48xx_0:TSOP45xx_0 TSOP48xx_1
 U 1 1 5AFDFBCA
 P 7450 5150
-F 0 "U1" H 6983 5200 50  0000 R CNN
+F 0 "TSOP48xx_1" H 6983 5200 50  0000 R CNN
 F 1 "TSOP45xx_0" H 6983 5109 50  0000 R CNN
 F 2 "Package_TO_SOT_THT:TO-220-3_Vertical" H 7400 4775 50  0001 C CNN

Commit message: Fixed layout, so the pinheader are on the correct side...
Parts:
- 433_RX1: footprint Package_TO_SOT_THT:TO-220-4_Vertical -> Sensors:RF_Receiver_433_MHz
- 433_TX1: footprint Package_TO_SOT_THT:TO-220-3_Vertical -> Sensors:RF_Transmitter_433_MHz
- CC1101: footprint cc1101:CC1101-868MHz-Module -> miscellaneous:CC1101-868MHz-Module
- C_0.22F1: footprint Capacitor_THT:CP_Radial_D10.0mm_P5.00mm -> Capacitor_THT:CP_Radial_D5.0mm_P2.50mm
- IR_D1: footprint Connector_PinHeader_2.54mm:PinHeader_1x02_P2.54mm_Vertical -> LED_THT:LED_D3.0mm_Horizontal_O6.35mm_Z10.0mm
- IR_D2: footprint Connector_PinHeader_2.54mm:PinHeader_1x02_P2.54mm_Vertical -> LED_THT:LED_D3.0mm_Horizontal_O6.35mm_Z10.0mm; footprint alternate (none) -> Connector_PinHeader_2.54mm:PinHeader_1x02_P2.54mm_Vertical
Changed lines of the file:
@@
 F 0 "IR_D1" H 5120 1470 50  0000 L CNN
 F 1 "IRL81A" H 5060 1290 50  0000 C CNN
-F 2 "Connector_PinHeader_2.54mm:PinHeader_1x02_P2.54mm_Vertical" H 5100 1575 50  0001 C CNN
+F 2 "LED_THT:LED_D3.0mm_Horizontal_O6.35mm_Z10.0mm" H 5100 1575 50  0001 C CNN
 F 3 "" H 5050 1400 50  0001 C CNN
 	1    5100 1400
@@
 F 0 "IR_D2" H 5620 1470 50  0000 L CNN
 F 1 "IRL81A" H 5560 1290 50  0000 C CNN
-F 2 "Connector_PinHeader_2.54mm:PinHeader_1x02_P2.54mm_Vertical" H 5600 1575 50  0001 C CNN
+F 2 "LED_THT:LED_D3.0mm_Horizontal_O6.35mm_Z10.0mm" H 5600 1575 50  0001 C CNN
 F 3 "" H 5550 1400 50  0001 C CNN
+F 4 "Connector_PinHeader_2.54mm:PinHeader_1x02_P2.54mm_Vertical" H 5600 1400 50  0001 C CNN "footprint alternate"
 	1    5600 1400
 	-1   0    0    -1
@@
 F 0 "CC1101" H 7041 6353 60  0000 L CNN
 F 1 "CC1101-868MHz-Module" H 7041 6247 60  0000 L CNN
-F 2 "cc1101:CC1101-868MHz-Module" H 5900 6300 60  0001 C CNN
+F 2 "miscellaneous:CC1101-868MHz-Module" H 5900 6300 60  0001 C CNN
 F 3 "" H 5900 6300 60  0001 C CNN
 	1    5900 6300
@@
 F 0 "C_0.22F1" H 8318 2146 50  0000 L CNN
 F 1 "0.22F" H 8318 2055 50  0000 L CNN
-F 2 "Capacitor_THT:CP_Radial_D10.0mm_P5.00mm" H 8238 1950 50  0001 C CNN
+F 2 "Capacitor_THT:CP_Radial_D5.0mm_P2.50mm" H 8238 1950 50  0001 C CNN
 F 3 "~" H 8200 2100 50  0001 C CNN
 	1    8200 2100
@@
 F 0 "433_TX1" H 7080 2742 50  0000 L CNN
 F 1 "433 MHz transmit" H 7080 2651 50  0000 L CNN
-F 2 "Package_TO_SOT_THT:TO-220-3_Vertical" H 7000 2700 50  0001 C CNN
+F 2 "Sensors:RF_Transmitter_433_MHz" H 7000 2700 50  0001 C CNN
 F 3 "~" H 7000 2700 50  0001 C CNN
 	1    7000 2700
@@
 F 0 "433_RX1" H 7079 2092 50  0000 L CNN
 F 1 "433 Mhz receive" H 7079 2001 50  0000 L CNN
-F 2 "Package_TO_SOT_THT:TO-220-4_Vertical" H 7000 2100 50  0001 C CNN
+F 2 "Sensors:RF_Receiver_433_MHz" H 7000 2100 50  0001 C CNN
 F 3 "~" H 7000 2100 50  0001 C CNN
 	1    7000 2100

Commit message: Prepared version 0.3.
Connections:
- wire segments 101 -> 102
Changed lines of the file:
@@
 	5950 1400 5950 1950
-Wire Wire Line
-	5000 1850 5000 3000
-Wire Wire Line
-	3150 1850 5000 1850
 Wire Wire Line
 	5000 3000 6800 3000
@@
 Wire Wire Line
 	6400 2000 6400 3100
-Connection ~ 3150 1850
 $Comp
 L ha_plattform-rescue:Raspberry_Pi_2_3 J3
@@
 Wire Wire Line
 	2550 5000 6400 5000
+Wire Wire Line
+	3050 1850 3050 1700
+Wire Wire Line
+	3050 1700 5000 1700
+Wire Wire Line
+	5000 1700 5000 3000
 $EndSCHEMATC
