File: nodemcu/nodemcu.sch (KiCad schematic (older format))
At the start: 2 parts

Commit message: Rerouted because footprints of 433mhz rx/tx were wrong-32-51.sch
Parts:
- gave numbers to parts that had none: 2
Changed lines of the file:
@@
 $EndDescr
 $Comp
-L nodemcu:NodeMCU_Amica_R2 U?
+L nodemcu:NodeMCU_Amica_R2 U1
 U 1 1 5B2FAF02
 P 1650 1750
-F 0 "U?" H 1650 2765 50  0000 C CNN
+F 0 "U1" H 1650 2765 50  0000 C CNN
 F 1 "NodeMCU_Amica_R2" H 1650 2674 50  0000 C CNN
 F 2 "nodemcu:NodeMCU_Amica_R2" H 1650 2583 50  0000 C CNN
@@
 $EndComp
 $Comp
-L nRF24L01+:nRF24L01+ U?
+L nRF24L01+:nRF24L01+ U2
 U 1 1 5B2FAF9E
 P 4100 1250
-F 0 "U?" H 4100 1765 50  0000 C CNN
+F 0 "U2" H 4100 1765 50  0000 C CNN
 F 1 "nRF24L01+" H 4100 1674 50  0000 C CNN
 F 2 "mysensors_radios:NRF24L01" H 4100 1350 50  0001 C CNN
